File: opm_coil_fork/final_coil_Z_testing_size.kicad_pcb (KiCad board)
At the start: 2 copper layers, 0 parts

Commit message: final windings for Z coil
Routing:
- net (no net): track 5297.7 -> 5838.2 mm, vias 0 -> 8
